Commit message: lecture_1_files

File: omtp_lecture_1/omtp course files lecture 1 (2023)/omtp_support/urdf/omtp.urdf (robot description, URDF)
Before this commit: robot omtp, 58 links, 57 joints
Links:
- removed link panda_3_hand
- removed link panda_3_leftfinger
- removed link panda_3_link0
- removed link panda_3_link1
- removed link panda_3_link2
- removed link panda_3_link3
- removed link panda_3_link4
- removed link panda_3_link5
- removed link panda_3_link6
- removed link panda_3_link7
- removed link panda_3_link8
- removed link panda_3_rightfinger
- removed link robot3_base
- removed link robot3_base_link
- removed link robot3_base_link_inertia
- removed link robot3_flange
- removed link robot3_forearm_link
- removed link robot3_pedestal_link
- removed link robot3_shoulder_link
- removed link robot3_tool0
- removed link robot3_upper_arm_link
- removed link robot3_wrist_1_link
- removed link robot3_wrist_2_link
- removed link robot3_wrist_3_link
Joints:
- removed joint panda_3_finger_joint1
- removed joint panda_3_finger_joint2
- removed joint panda_3_hand_joint
- removed joint panda_3_joint1
- removed joint panda_3_joint2
- removed joint panda_3_joint3
- removed joint panda_3_joint4
- removed joint panda_3_joint5
- removed joint panda_3_joint6
- removed joint panda_3_joint7
- removed joint panda_3_joint8
- removed joint panda_3_virtual_joint
- removed joint robot3-robot3_pedestal_joint
- removed joint robot3_base_link-base_fixed_joint
- removed joint robot3_base_link-base_link_inertia
- removed joint robot3_elbow_joint
- removed joint robot3_flange-tool0
- removed joint robot3_pedestal_joint
- removed joint robot3_shoulder_lift_joint
- removed joint robot3_shoulder_pan_joint
- removed joint robot3_wrist_1_joint
- removed joint robot3_wrist_2_joint
- removed joint robot3_wrist_3-flange
- removed joint robot3_wrist_3_joint

File: omtp_lecture_1/omtp course files lecture 1 (2023)/omtp_support/urdf/omtp_factory.xacro (robot description, xacro)
@@ -29,22 +29,24 @@
   <xacro:panda_arm arm_id="$(arg arm_id_1)" connected_to="robot1_pedestal_link"  xyz="0 0 0.95" safety_distance="0.03"/>
   <xacro:hand ns="$(arg arm_id_1)" rpy="0 0 ${-pi/4}" connected_to="$(arg arm_id_1)_link8" safety_distance="0.03"/>
-  <!-- dual arm -->
+  <!-- Gazebo control -->
+  <xacro:include filename="$(find franka_description)/robots/panda.gazebo.xacro"/>
+  <xacro:include filename="$(find franka_description)/robots/panda.control.xacro"/>
+  <!-- Panda 1 gazebo -->
+  <!--     arm     -->
+  <xacro:arm_gazebo arm_id="$(arg arm_id_1)"/>
+  <xacro:arm_control arm_id="$(arg arm_id_1)"/>
+  <!--     hand    -->
+  <xacro:hand_gazebo arm_id="$(arg arm_id_1)"/>
+  <xacro:hand_control arm_id="$(arg arm_id_1)"/>
+  <!-- dual arm
   <xacro:arg name="arm_id_3" default="panda_3" />
   <xacro:arg name="arm_id_4" default="panda_4" />
   <xacro:include filename="$(find franka_description)/robots/panda_arm.xacro"/>
   <xacro:include filename="$(find franka_description)/robots/hand.xacro"/>
-  <!-- Panda 1 arm with gripper -->
+  -->
+  <!-- Panda 2 arm with gripper
   <xacro:panda_arm arm_id="$(arg arm_id_3)" connected_to="robot2_pedestal_link"  xyz="0 0 0.95" safety_distance="0.03"/>
   <xacro:hand ns="$(arg arm_id_3)" rpy="0 0 ${-pi/4}" connected_to="$(arg arm_id_3)_link8" safety_distance="0.03"/>
-  <!-- ==================================================== -->
-  <!-- UR robots -->
-  <!-- ==================================================== -->
-  <xacro:include filename="$(find ur_description)/urdf/inc/ur5_macro.xacro"/>
-  <xacro:ur5_robot prefix="robot3_"/>
-  <joint name="robot3-robot3_pedestal_joint" type="fixed">
-    <parent link="robot3_pedestal_link"/>
-    <child link="robot3_base_link"/>
-    <origin xyz="0 0 0.95" rpy="0 0 ${-pi/4}"/>
-  </joint>
+  -->
   <!-- ==================================================== -->
   <!-- Robot 1,2 pedestal -->
@@ -56,7 +58,4 @@
   <xacro:robot_pedestal_urdf pedestal_prefix="robot2_" pedestal_parent="world_interface" pedestal_height="0.95">
     <origin xyz="-3.6 7.6 0.0" rpy="0 0 0"/>
-  </xacro:robot_pedestal_urdf>
-  <xacro:robot_pedestal_urdf pedestal_prefix="robot3_" pedestal_parent="world_interface" pedestal_height="0.95">
-    <origin xyz="-1.5 8 0.0" rpy="0 0 0"/>
   </xacro:robot_pedestal_urdf>
   <!-- ==================================================== -->
