Commit message: lecture_2 finished
two arm in gazebo working , pick and place python code written

File: Week_1/omtp_w1/omtp_support/urdf/omtp.urdf (robot description, URDF)
Before this commit: robot omtp, 46 links, 45 joints
Links:
- removed link panda_3_hand
- removed link panda_3_leftfinger
- removed link panda_3_link0
- removed link panda_3_link1
- removed link panda_3_link2
- removed link panda_3_link3
- removed link panda_3_link4
- removed link panda_3_link5
- removed link panda_3_link6
- removed link panda_3_link7
- removed link panda_3_link8
- removed link panda_3_rightfinger
- added link bottle_1bottle, mass 10; collision mesh filename=package://omtp_support/meshes/bottle/beer_bottle.dae; visual mesh filename=package://omtp_support/meshes/bottle/beer_bottle.dae
- added link bottle_2bottle, mass 10; collision mesh filename=package://omtp_support/meshes/bottle/beer_bottle.dae; visual mesh filename=package://omtp_support/meshes/bottle/beer_bottle.dae
- added link bottle_3bottle, mass 10; collision mesh filename=package://omtp_support/meshes/bottle/beer_bottle.dae; visual mesh filename=package://omtp_support/meshes/bottle/beer_bottle.dae
- added link bottle_4bottle, mass 10; collision mesh filename=package://omtp_support/meshes/bottle/beer_bottle.dae; visual mesh filename=package://omtp_support/meshes/bottle/beer_bottle.dae
- added link panda_2_hand, mass 0.48; collision mesh filename=package://franka_description/meshes/collision/hand.stl; visual mesh filename=package://franka_description/meshes/visual/hand.dae
- added link panda_2_leftfinger, mass 0.1; collision mesh filename=package://franka_description/meshes/collision/finger.stl; visual mesh filename=package://franka_description/meshes/visual/finger.dae
- added link panda_2_link0, mass 3.06; collision mesh filename=package://franka_description/meshes/collision/link0.stl; visual mesh filename=package://franka_description/meshes/visual/link0.dae
- added link panda_2_link1, mass 2.34; collision mesh filename=package://franka_description/meshes/collision/link1.stl; visual mesh filename=package://franka_description/meshes/visual/link1.dae
- added link panda_2_link2, mass 2.36; collision mesh filename=package://franka_description/meshes/collision/link2.stl; visual mesh filename=package://franka_description/meshes/visual/link2.dae
- added link panda_2_link3, mass 2.38; collision mesh filename=package://franka_description/meshes/collision/link3.stl; visual mesh filename=package://franka_description/meshes/visual/link3.dae
- added link panda_2_link4, mass 2.43; collision mesh filename=package://franka_description/meshes/collision/link4.stl; visual mesh filename=package://franka_description/meshes/visual/link4.dae
- added link panda_2_link5, mass 3.5; collision mesh filename=package://franka_description/meshes/collision/link5.stl; visual mesh filename=package://franka_description/meshes/visual/link5.dae
- added link panda_2_link6, mass 1.47; collision mesh filename=package://franka_description/meshes/collision/link6.stl; visual mesh filename=package://franka_description/meshes/visual/link6.dae
- added link panda_2_link7, mass 0.45; collision mesh filename=package://franka_description/meshes/collision/link7.stl; visual mesh filename=package://franka_description/meshes/visual/link7.dae
- added link panda_2_link8, mass 0.0
- added link panda_2_rightfinger, mass 0.1; collision mesh filename=package://franka_description/meshes/collision/finger.stl; visual mesh filename=package://franka_description/meshes/visual/finger.dae
- link festo_straight_4festo_module: geometry collision mesh filename=package://aau_lab_ros_models/meshes/festo_t_module/festo_t_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; visual mesh filename=package://aau_lab_ros_models/meshes/festo_t_module/festo_t_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
- link panda_1_hand: mass None -> 0.48; geometry collision mesh filename=package://franka_description/meshes/collision/hand.stl; visual mesh filename=package://franka_description/meshes/visual/hand.dae
- link panda_1_leftfinger: mass None -> 0.1; geometry collision mesh filename=package://franka_description/meshes/collision/finger.stl; visual mesh filename=package://franka_description/meshes/visual/finger.dae
- link panda_1_link0: mass None -> 3.06; geometry collision mesh filename=package://franka_description/meshes/collision/link0.stl; visual mesh filename=package://franka_description/meshes/visual/link0.dae
- link panda_1_link1: mass None -> 2.34; geometry collision mesh filename=package://franka_description/meshes/collision/link1.stl; visual mesh filename=package://franka_description/meshes/visual/link1.dae
- link panda_1_link2: mass None -> 2.36; geometry collision mesh filename=package://franka_description/meshes/collision/link2.stl; visual mesh filename=package://franka_description/meshes/visual/link2.dae
- link panda_1_link3: mass None -> 2.38; geometry collision mesh filename=package://franka_description/meshes/collision/link3.stl; visual mesh filename=package://franka_description/meshes/visual/link3.dae
- link panda_1_link4: mass None -> 2.43; geometry collision mesh filename=package://franka_description/meshes/collision/link4.stl; visual mesh filename=package://franka_description/meshes/visual/link4.dae
- link panda_1_link5: mass None -> 3.5; geometry collision mesh filename=package://franka_description/meshes/collision/link5.stl; visual mesh filename=package://franka_description/meshes/visual/link5.dae
- link panda_1_link6: mass None -> 1.47; geometry collision mesh filename=package://franka_description/meshes/collision/link6.stl; visual mesh filename=package://franka_description/meshes/visual/link6.dae
- link panda_1_link7: mass None -> 0.45; geometry collision mesh filename=package://franka_description/meshes/collision/link7.stl; visual mesh filename=package://franka_description/meshes/visual/link7.dae
- link panda_1_link8: mass None -> 0.0; geometry 
- link panda_1_rightfinger: mass None -> 0.1; geometry collision mesh filename=package://franka_description/meshes/collision/finger.stl; visual mesh filename=package://franka_description/meshes/visual/finger.dae
Joints:
- removed joint panda_3_finger_joint1
- removed joint panda_3_finger_joint2
- removed joint panda_3_hand_joint
- removed joint panda_3_joint1
- removed joint panda_3_joint2
- removed joint panda_3_joint3
- removed joint panda_3_joint4
- removed joint panda_3_joint5
- removed joint panda_3_joint6
- removed joint panda_3_joint7
- removed joint panda_3_joint8
- removed joint panda_3_virtual_joint
- added joint bottle_1bottle_interface: type fixed, parent world_interface, child bottle_1bottle, origin xyz=-3.0 8.3 0.95 rpy=0 0 0
- added joint bottle_2bottle_interface: type fixed, parent world_interface, child bottle_2bottle, origin xyz=-3.0 9.3 0.95 rpy=0 0 0
- added joint bottle_3bottle_interface: type fixed, parent world_interface, child bottle_3bottle, origin xyz=-3.0 11.4 0.95 rpy=0 0 0
- added joint bottle_4bottle_interface: type fixed, parent world_interface, child bottle_4bottle, origin xyz=-3.0 11.7 0.95 rpy=0 0 0
- added joint panda_2_finger_joint1: type prismatic, parent panda_2_hand, child panda_2_leftfinger, origin xyz=0 0 0.0584 rpy=0 0 0, axis 0 1 0, limit lower=0.0 upper=0.04 effort=150 velocity=0.2
- added joint panda_2_finger_joint2: type prismatic, parent panda_2_hand, child panda_2_rightfinger, origin xyz=0 0 0.0584 rpy=0 0 0, axis 0 -1 0, limit lower=0.0 upper=0.04 effort=150 velocity=0.2
- added joint panda_2_hand_joint: type fixed, parent panda_2_link8, child panda_2_hand, origin xyz=0 0 0 rpy=0 0 -0.785398163397
- added joint panda_2_joint1: type revolute, parent panda_2_link0, child panda_2_link1, origin xyz=0 0 0.333 rpy=0 0 0, axis 0 0 1, limit lower=-2.8973 upper=2.8973 effort=87 velocity=2.175
- added joint panda_2_joint2: type revolute, parent panda_2_link1, child panda_2_link2, origin xyz=0 0 0 rpy=-1.57079632679 0 0, axis 0 0 1, limit lower=-1.7628 upper=1.7628 effort=87 velocity=2.175
- added joint panda_2_joint3: type revolute, parent panda_2_link2, child panda_2_link3, origin xyz=0 -0.316 0 rpy=1.57079632679 0 0, axis 0 0 1, limit lower=-2.8973 upper=2.8973 effort=87 velocity=2.175
- added joint panda_2_joint4: type revolute, parent panda_2_link3, child panda_2_link4, origin xyz=0.0825 0 0 rpy=1.57079632679 0 0, axis 0 0 1, limit lower=-3.0718 upper=-0.0698 effort=87 velocity=2.175
- added joint panda_2_joint5: type revolute, parent panda_2_link4, child panda_2_link5, origin xyz=-0.0825 0.384 0 rpy=-1.57079632679 0 0, axis 0 0 1, limit lower=-2.8973 upper=2.8973 effort=12 velocity=2.61
- added joint panda_2_joint6: type revolute, parent panda_2_link5, child panda_2_link6, origin xyz=0 0 0 rpy=1.57079632679 0 0, axis 0 0 1, limit lower=-0.0175 upper=3.7525 effort=12 velocity=2.61
- added joint panda_2_joint7: type revolute, parent panda_2_link6, child panda_2_link7, origin xyz=0.088 0 0 rpy=1.57079632679 0 0, axis 0 0 1, limit lower=-2.8973 upper=2.8973 effort=12 velocity=2.61
- added joint panda_2_joint8: type fixed, parent panda_2_link7, child panda_2_link8, origin xyz=0 0 0.107 rpy=0 0 0, axis 0 0 0
- added joint panda_2_virtual_joint: type fixed, parent robot2_pedestal_link, child panda_2_link0, origin xyz=0 0 0.95 rpy=0 0 0
- joint festo_straight_1festo_module_to_world_interface: origin xyz=-1.84 7.0 0.0 rpy=0 0 -1.57079632679 -> xyz=-3.0 8.0 0.0 rpy=0 0 0
- joint festo_straight_2festo_module_to_world_interface: origin xyz=-3.0 8.0 0.0 rpy=0 0 0 -> xyz=-3.0 9.15 0.0 rpy=0 0 0
- joint festo_straight_3festo_module_to_world_interface: origin xyz=-3.0 9.15 0.0 rpy=0 0 0 -> xyz=-3.0 10.30 0.0 rpy=0 0 0
- joint festo_straight_4festo_module_to_world_interface: origin xyz=-3.0 10.30 0.0 rpy=0 0 0 -> xyz=-1.84 7.0 0.0 rpy=0 0 -1.57079632679
- joint panda_1_finger_joint2: mimic joint=panda_1_finger_joint1 -> (none)
