Commit message: grasping

File: omtp_lecture5/urdf/omtp_panda5.urdf.xacro (robot description, xacro)
@@ -142,5 +142,5 @@
   <joint name="camera_joint" type="fixed">
     <axis xyz="0 1 0" />
-    <origin xyz="0.0 11.25 2.0" rpy="0 1.57079 0"/>
+    <origin xyz="0.0 11.25 1.6" rpy="0 1.57079 0"/>
     <parent link="world"/>
     <child link="camera_link"/>
